File: IR_Sense.kicad_pcb (KiCad board)
At the start: 2 copper layers, 29.7 x 18.2 mm, 17 parts, among them J1 Conn_01x03, J2 Conn_01x02, Q1 VEMT2020X01, U2 LMV321

Commit message: new values
Parts:
- R3: value 5k -> 150k
- R5, R8: value 3k -> 100k
- R6: value 66k -> 470k
- R7: value 5.6k -> 100k
Changed lines of the file:
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@@
 			)
 		)
-		(property "Value" "66k"
+		(property "Value" "470k"
 			(at 0 1.43 0)
 			(layer "F.Fab")
@@
 			)
 		)
-		(property "Value" "3k"
+		(property "Value" "100k"
 			(at 0 1.43 135)
 			(layer "F.Fab")
@@
 			)
 		)
-		(property "Value" "3k"
+		(property "Value" "100k"
 			(at 0 1.43 90)
 			(layer "F.Fab")
@@
 			)
 		)
-		(property "Value" "5.6k"
+		(property "Value" "100k"
 			(at 0 1.43 0)
 			(layer "F.Fab")
@@
 			)
 		)
-		(property "Value" "5k"
+		(property "Value" "150k"
 			(at -0.000001 1.429998 0)
 			(layer "F.Fab")
