File: IR_Sense.kicad_sch (KiCad schematic)
At the start: 15 parts, among them J1 Conn_01x03, J2 Conn_01x02, Q1 VEMT2020X01, U2 LMV321

Commit message: new values
Parts:
- R3: value 5k -> 150k
- R5, R8: value 3k -> 100k
- R6: value 66k -> 470k
- R7: value 5.6k -> 100k
Changed lines of the file:
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@@
 			)
 		)
-		(property "Value" "3k"
+		(property "Value" "100k"
 			(at 137.16 51.816 90)
 			(effects
@@
 			)
 		)
-		(property "Value" "5.6k"
+		(property "Value" "100k"
 			(at 140.716 67.564 90)
 			(effects
@@
 			)
 		)
-		(property "Value" "5k"
-			(at 115.824 46.736 0)
+		(property "Value" "150k"
+			(at 114.3 46.99 0)
 			(effects
 				(font
@@
 			)
 		)
-		(property "Value" "66k"
+		(property "Value" "470k"
 			(at 153.67 41.656 90)
 			(effects
@@
 			)
 		)
-		(property "Value" "3k"
+		(property "Value" "100k"
 			(at 140.716 79.756 90)
 			(effects
