File: IR_Sense.kicad_sch (KiCad schematic)
At the start: 15 parts, among them J1 Conn_01x03, J2 Conn_01x02, Q1 VEMT2020X01, U2 LMV321

Commit message: SSL27 refurbish
Parts:
- J1: footprint IR_Sense:J1-SMD_PADS_ONLY -> lcsc:CONN-SMD_3P-P1.25_XUNPU_WAFER-MX1.25-3PCB
- J2: footprint IR_Sense:Tx_Power_Pads -> lcsc:CONN-SMD_2P-P1.25_WAFER-MX1.25-2PCB
- R3: value 150k -> 32k
- R5, R8: value 100k -> 3k
- R6: value 470k -> 66k
- R7: value 100k -> 5.6k
Connections:
- net GND: no longer H1.1, H2.1, H3.1, H4.1
- no-connect marks 0 -> 4
