File: .history/IR_Sense.kicad_pcb (KiCad board)
At the start: 2 copper layers, 39.7 x 18.2 mm, 17 parts, among them J1 Conn_01x03, J2 Conn_01x02, Q1 VEMT2020X01, U2 LMV321

Commit message: Align amplifier resistors with 2026 tested new values, pending inspection
Parts:
- R3: value 32k -> 150K
- R5, R8: value 3k -> 100k
- R6: value 66k -> 470k
- R7: value 5.6k -> 100k
Changed lines of the file:
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@@
 			)
 		)
-		(property "Value" "66k"
+		(property "Value" "470k"
 			(at 0 1.43 0)
 			(layer "F.Fab")
@@
 			)
 		)
-		(property "Value" "3k"
+		(property "Value" "100k"
 			(at 0 1.430001 0)
 			(layer "F.Fab")
@@
 			)
 		)
-		(property "Value" "3k"
+		(property "Value" "100k"
 			(at 0 1.43 90)
 			(layer "F.Fab")
@@
 			)
 		)
-		(property "Value" "5.6k"
+		(property "Value" "100k"
 			(at 0 1.43 0)
 			(layer "F.Fab")
@@
 			)
 		)
-		(property "Value" "32k"
+		(property "Value" "150K"
 			(at -0.000001 1.429998 110)
 			(layer "F.Fab")

Commit message: 增大光感元器件焊盘 size，添加信号外部 test point
Parts:
- R1, R3, R5, R6, R7, R8: footprint Resistor_SMD:R_0603_1608Metric_Pad0.98x0.95mm_HandSolder -> Resistor_SMD:R_0603_1608Metric
- moved G*** 2.21 mm to (83.5, 74.4)
- moved G*** 1.22 mm to (105.7, 74.9)
Routing:
- net IR I/O: track 6.34 -> 8.62 mm, vias 0 -> 1
- net GND: vias 19 -> 20
Other:
- board text added: "IR"
- board text removed: "IRD"
