File: .history/IR_Sense.kicad_sch (KiCad schematic)
At the start: 15 parts, among them J1 Conn_01x03, J2 Conn_01x02, Q1 VEMT2020X01, U2 LMV321

Commit message: Align amplifier resistors with 2026 tested new values, pending inspection
Parts:
- R3: value 32k -> 150K
- R5, R8: value 3k -> 100k
- R6: value 66k -> 470k
- R7: value 5.6k -> 100k
Changed lines of the file:
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@@
 			)
 		)
-		(property "Value" "3k"
+		(property "Value" "100k"
 			(at 137.16 51.816 90)
 			(show_name no)
@@
 			)
 		)
-		(property "Value" "5.6k"
+		(property "Value" "100k"
 			(at 140.716 67.564 90)
 			(show_name no)
@@
 			)
 		)
-		(property "Value" "32k"
+		(property "Value" "150K"
 			(at 115.824 46.736 0)
 			(show_name no)
@@
 			)
 		)
-		(property "Value" "66k"
+		(property "Value" "470k"
 			(at 153.67 41.656 90)
 			(show_name no)
@@
 			)
 		)
-		(property "Value" "3k"
+		(property "Value" "100k"
 			(at 140.716 79.756 90)
 			(show_name no)

Commit message: 增大光感元器件焊盘 size，添加信号外部 test point
Parts:
- R1, R3, R5, R6, R7, R8: footprint Resistor_SMD:R_0603_1608Metric_Pad0.98x0.95mm_HandSolder -> Resistor_SMD:R_0603_1608Metric
Changed lines of the file:
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@@
 			)
 		)
-		(property "Footprint" "Resistor_SMD:R_0603_1608Metric_Pad0.98x0.95mm_HandSolder"
+		(property "Footprint" "Resistor_SMD:R_0603_1608Metric"
 			(at 52.832 73.66 90)
 			(hide yes)
@@
 			)
 		)
-		(property "Footprint" "Resistor_SMD:R_0603_1608Metric_Pad0.98x0.95mm_HandSolder"
+		(property "Footprint" "Resistor_SMD:R_0603_1608Metric"
 			(at 137.16 56.388 90)
 			(hide yes)
@@
 			)
 		)
-		(property "Footprint" "Resistor_SMD:R_0603_1608Metric_Pad0.98x0.95mm_HandSolder"
+		(property "Footprint" "Resistor_SMD:R_0603_1608Metric"
 			(at 140.208 67.31 90)
 			(hide yes)
@@
 			)
 		)
-		(property "Footprint" "Resistor_SMD:R_0603_1608Metric_Pad0.98x0.95mm_HandSolder"
+		(property "Footprint" "Resistor_SMD:R_0603_1608Metric"
 			(at 118.872 45.72 90)
 			(hide yes)
@@
 			)
 		)
-		(property "Footprint" "Resistor_SMD:R_0603_1608Metric_Pad0.98x0.95mm_HandSolder"
+		(property "Footprint" "Resistor_SMD:R_0603_1608Metric"
 			(at 153.67 46.228 90)
 			(hide yes)
@@
 			)
 		)
-		(property "Footprint" "Resistor_SMD:R_0603_1608Metric_Pad0.98x0.95mm_HandSolder"
+		(property "Footprint" "Resistor_SMD:R_0603_1608Metric"
 			(at 140.208 80.01 90)
 			(hide yes)
